Commit message: working prototype with modified panda urdf

File: robots/panda/robot.urdf (robot description, URDF)
Before this commit: robot panda, 8 links, 7 joints
Joints:
- joint panda_joint1: limit lower=-2.8973 upper=2.8973 effort=87.0 velocity=2.175 -> lower=-20.8973 upper=20.8973 effort=87.0 velocity=2.175
- joint panda_joint2: limit lower=-1.7628 upper=1.7628 effort=87.0 velocity=2.175 -> lower=-10.7628 upper=10.7628 effort=87.0 velocity=2.175
- joint panda_joint6: limit lower=-0.0175 upper=3.7525 effort=12.0 velocity=2.61 -> lower=-10.0175 upper=3.7525 effort=12.0 velocity=2.61
